File: MRCS-Adapter-CRMI8-RJ45-Inverting.brd (EAGLE design)
At the start: 31 x 64 mm, 18 parts, among them IC1 74LS540N, J1 RJ45, M1 MOUNTINGHOLE, M2 MOUNTINGHOLE, M3 MOUNTINGHOLE

Commit message: various adjustments
minor board layout adjustments
Parts:
- added RN1: 4.7K, resistor-sil:SIL9
- moved IC1 10.8 mm to (15.9, 37.5)
- moved J1 10.8 mm to (16.8, 69.5)
- moved J4 10.8 mm to (3.81, 60.1)
- moved M1 10.8 mm to (16.5, 69.5)
- moved R1 10.8 mm to (26.0, 51.4)
- moved R2 10.8 mm to (23.5, 51.4)
- moved R3 10.8 mm to (21.0, 51.4)
- moved R4 10.8 mm to (18.4, 51.4)
- moved R5 10.8 mm to (15.9, 51.4)
- moved R6 10.8 mm to (13.3, 51.4)
- moved R7 10.8 mm to (10.8, 51.4)
- moved R8 10.8 mm to (8.26, 51.4)
- moved U$1 10.8 mm to (16.5, 69.5)
- moved M2 1.90 mm to (27.3, 20.0)
- moved M3 1.90 mm to (3.17, 20.0)
Connections:
- net L1: now also RN1.9
- net L2: now also RN1.8
- net L3: now also RN1.7
- net L4: now also RN1.6
- net L5: now also RN1.5
- net L6: now also RN1.4
- net L7: now also RN1.3
- net L8: now also RN1.2
- net VCC: now also RN1.1
Routing:
- net VCC: track 34.0 -> 52.0 mm
- net L2: track 17.7 -> 35.1 mm
- net L7: track 18.0 -> 28.8 mm
- net L6: track 17.1 -> 27.9 mm
- net L4: track 16.5 -> 27.3 mm
- net L3: track 17.1 -> 27.9 mm
- net L1: track 19.3 -> 30.1 mm
- net L8: track 19.6 -> 30.4 mm
- net L5: track 16.7 -> 27.5 mm
Other:
- board size 31 x 64 mm -> 31 x 74.8 mm
