File: MRCS-Adapter-CRMI8-RJ45-Inverting.brd (EAGLE design)
At the start: 31 x 74.8 mm, 20 parts, among them IC1 74LS540N, J1 RJ45, M1 MOUNTINGHOLE, M2 MOUNTINGHOLE, M3 MOUNTINGHOLE

Commit message: Minor label changes
the Claifornia Prop 65 warning covered the cuttable links under the limiting resistor pads, so I moved them and deleted some of John's SPCoast comments.  It is important that the user can see the links to cut them.
Parts:
- added U$3: (no value), MRCSLogoBtm:MRCSLOGOBTM
- moved U$2 33.0 mm to (18.4, 17.8)
Other:
- board text added: "CMRI Inverting RJ45 Breakout"
- board text added: "CMRI RJ45 Inverting"
- board text removed: "Breakout"
- board text removed: "CMRI Accessory"
- board text removed: "Made in the PCR, Coast Division, NMRA"
- board text removed: "Model Railroading is fun!"
- board text removed: "RJ45"
- board text removed: "SPCoast"
- board text removed: "www . SPCoast . com"
Changed lines of the file:
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@@
 <layer number="50" name="dxf" color="7" fill="1" visible="no" active="yes"/>
 <layer number="51" name="tDocu" color="51" fill="1" visible="yes" active="yes"/>
-<layer number="52" name="bDocu" color="15" fill="1" visible="no" active="yes"/>
+<layer number="52" name="bDocu" color="15" fill="1" visible="yes" active="yes"/>
 <layer number="53" name="tGND_GNDA" color="7" fill="9" visible="no" active="no"/>
 <layer number="54" name="bGND_GNDA" color="1" fill="9" visible="no" active="no"/>
@@
 <text x="29.3624" y="30.1752" size="1.778" layer="51" font="vector" rot="SR90">CMRI8-RJ45 Inverting Adapter</text>
 <text x="0.635" y="16.383" size="1.016" layer="51" font="vector" rot="SR0">v1.0</text>
-<text x="28.5158" y="14.6744" size="0.8128" layer="52" font="vector" rot="SMR0">Made in the PCR, Coast Division, NMRA</text>
 <text x="18.538" y="45.444" size="0.8128" layer="52" font="vector" rot="SMR0">Solder
 Side</text>
-<text x="22.5568" y="16.1382" size="0.8128" layer="52" font="vector" ratio="15" rot="SMR0">www . SPCoast . com</text>
-<text x="20.3639" y="37.9406" size="0.8128" layer="52" font="vector" ratio="15" rot="MR0">CMRI Accessory</text>
-<text x="24.018" y="34.249" size="2.54" layer="52" font="vector" ratio="20" rot="SMR0">Breakout</text>
-<text x="23.9692" y="17.3851" size="0.8128" layer="52" font="vector" rot="SMR0">Model Railroading is fun!</text>
-<text x="19.827" y="41.345" size="2.54" layer="52" font="vector" ratio="20" rot="SMR0">RJ45</text>
+<text x="25.4439" y="39.2106" size="0.8128" layer="52" font="vector" ratio="15" rot="MR0">CMRI Inverting RJ45 Breakout</text>
+<text x="29.987" y="42.615" size="1.778" layer="52" font="vector" ratio="20" rot="SMR0">CMRI RJ45 Inverting</text>
 <text x="0.635" y="18.923" size="1.016" layer="51" font="vector" rot="SR0">2020.11</text>
-<text x="22.971" y="43.815" size="1.016" layer="52" font="vector" rot="SMR270">SPCoast</text>
 <text x="1.651" y="12.065" size="1.016" layer="51" font="vector" rot="SR0">3.5mm</text>
 <text x="26.67" y="2.159" size="1.016" layer="51" font="vector" rot="SR0">0.156</text>
@@
 <attribute name="MF" value="" x="14.605" y="26.67" size="1.778" layer="27" font="vector" ratio="10" display="off"/>
 </element>
-<element name="U$2" library="MRCS-prop65warningBtm" package="CA-PROP65WARNING" value="" x="19.685" y="50.8"/>
+<element name="U$2" library="MRCS-prop65warningBtm" package="CA-PROP65WARNING" value="" x="18.415" y="17.78"/>
+<element name="U$3" library="MRCSLogoBtm" package="MRCSLOGOBTM" value="" x="1.27" y="49.53"/>
 </elements>
 <signals>
